Commit message: After Dockerising1

File: src/dual_arm_description/urdf/dual_ur5.urdf.xacro (robot description, xacro)
@@ -8,6 +8,6 @@
         <box size="0.4 1.0 0.8"/>
       </geometry>
-      <material name="dark_grey">
-        <color rgba="0.3 0.3 0.3 1.0"/>
+      <material name="dark_blue">
+        <color rgba="0.1 0.2 0.4 1.0"/>
       </material>
     </visual>
